File: _autosave-TIME II PCB.kicad_pcb (KiCad board)
At the start: 2 copper layers, 70 x 50 mm, 77 parts, among them J1 USB_C_Receptacle, J2 SD_Card, J4 Conn_01x06, J5 Conn_01x06, J6 Conn_01x06, J7 Conn_01x02_Male, J8 Conn_01x02_Male, Q1 VNP10N07, Q4 VNP10N07, Q5 VNP10N07, SW3 SW_SPDT, U2 ADP2303, U3 LTC4420CMSE-PBF, U7 STM32F103C8Tx, Y1 16 khz

Commit message: update
Parts:
- C11, R28: moved to F.Cu
- moved C11 19.9 mm to (196.8, 79.8), turned to 90 degrees
- moved R28 5.44 mm to (194.5, 78.5)
Routing:
- net BAT: track 37.2 -> 5.43 mm, vias 3 -> 0
- net 5v: track 253.7 -> 245.9 mm, vias 6 -> 5
- net GND: track 84.0 -> 86.6 mm
- net BAT_REAL: track 2.66 -> 0.33 mm
