File: _autosave-TIME II PCB.kicad_sch (KiCad schematic)
At the start: 77 parts, among them J1 USB_C_Receptacle, J2 SD_Card, J4 Conn_01x06, J5 Conn_01x06, J6 Conn_01x06, J7 Conn_01x02_Male, J8 Conn_01x02_Male, Q1 VNP10N07, Q4 VNP10N07, Q5 VNP10N07, SW3 SW_SPDT, U2 ADP2303, U3 LTC4420CMSE-PBF, U7 STM32F103C8Tx, Y1 16 khz

Commit message: update
Parts:
- added R13, R18, R5: R, symbol Device:R
Connections:
- net heater_1: now also R5.1; no longer Q4.1 (G)
- net heater_2: now also R13.1; no longer Q1.1 (G)
- net heater_3: now also R18.1; no longer Q5.1 (G)
- new net: Q1.1 (G), R13.2
- new net: Q5.1 (G), R18.2
Changed lines of the file:
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@@
+    (stroke (width 0) (type default))
+  )
+  (wire (pts (xy 389.89 157.48) (xy 392.43 157.48))
     (stroke (width 0) (type default))
   )
@@
     (stroke (width 0) (type default))
   )
+  (wire (pts (xy 379.73 157.48) (xy 382.27 157.48))
+    (stroke (width 0) (type default))
+  )
   (wire (pts (xy 480.06 240.03) (xy 483.87 240.03))
     (stroke (width 0) (type default))
@@
     (stroke (width 0) (type default))
   )
-  (wire (pts (xy 379.73 157.48) (xy 392.43 157.48))
-    (stroke (width 0) (type default))
-  )
   (wire (pts (xy 200.66 246.38) (xy 205.74 246.38))
     (stroke (width 0) (type default))
@@
     (stroke (width 0) (type default))
   )
-  (wire (pts (xy 452.12 135.89) (xy 464.82 135.89))
-    (stroke (width 0) (type default))
-  )
   (wire (pts (xy 457.2 106.68) (xy 464.82 106.68))
     (stroke (width 0) (type default))
@@
     (stroke (width 0) (type default))
   )
+  (wire (pts (xy 384.81 106.68) (xy 387.35 106.68))
+    (stroke (width 0) (type default))
+  )
   (wire (pts (xy 85.09 74.93) (xy 88.9 74.93))
     (stroke (width 0) (type default))
@@
     (stroke (width 0) (type default))
   )
+  (wire (pts (xy 452.12 135.89) (xy 454.66 135.89))
+    (stroke (width 0) (type default))
+  )
   (wire (pts (xy 111.76 243.84) (xy 111.76 254))
     (stroke (width 0) (type default))
@@
     (stroke (width 0) (type default))
   )
+  (wire (pts (xy 462.28 135.89) (xy 464.82 135.89))
+    (stroke (width 0) (type default))
+  )
   (wire (pts (xy 109.22 264.16) (xy 104.14 264.16))
     (stroke (width 0) (type default))
@@
     (stroke (width 0) (type default))
   )
-  (wire (pts (xy 384.81 106.68) (xy 397.51 106.68))
-    (stroke (width 0) (type default))
-  )
   (wire (pts (xy 332.74 40.64) (xy 332.74 43.18))
     (stroke (width 0) (type default))
@@
   )
   (polyline (pts (xy 246.38 200.66) (xy 63.5 200.66))
+    (stroke (width 0) (type default))
+  )
+  (wire (pts (xy 397.51 106.68) (xy 398.78 106.68))
     (stroke (width 0) (type default))
   )
@@
     )
   )
+  (symbol (lib_id "Device:R") (at 458.47 135.89 90) (unit 1)
+    (in_bom yes) (on_board yes) (dnp no) (fields_autoplaced)
+    (property "Reference" "R18" (at 458.47 129.54 90)
+      (effects (font (size 1.27 1.27)))
+    )
+    (property "Value" "R" (at 458.47 132.08 90)
+      (effects (font (size 1.27 1.27)))
+    )
+    (property "Footprint" "" (at 458.47 137.668 90)
+      (effects (font (size 1.27 1.27)) hide)
+    )
+    (property "Datasheet" "~" (at 458.47 135.89 0)
+      (effects (font (size 1.27 1.27)) hide)
+    )
+    (pin "1")
+    (pin "2")
+    (instances
+      (project "TIME II PCB"
+        (path "/ada74dd6-9313-41da-aa43-aea44c6d55c8"
+          (reference "R18") (unit 1)
+        )
+      )
+    )
+  )
   (symbol (lib_id "Device:C") (at 81.28 245.11 0) (unit 1)
     (in_bom yes) (on_board yes) (dnp no) (fields_autoplaced)
@@
     )
   )
+  (symbol (lib_id "Device:R") (at 386.08 157.48 90) (unit 1)
+    (in_bom yes) (on_board yes) (dnp no) (fields_autoplaced)
+    (property "Reference" "R13" (at 386.08 151.13 90)
+      (effects (font (size 1.27 1.27)))
+    )
+    (property "Value" "R" (at 386.08 153.67 90)
+      (effects (font (size 1.27 1.27)))
+    )
+    (property "Footprint" "" (at 386.08 159.258 90)
+      (effects (font (size 1.27 1.27)) hide)
+    )
+    (property "Datasheet" "~" (at 386.08 157.48 0)
+      (effects (font (size 1.27 1.27)) hide)
+    )
+    (pin "1")
+    (pin "2")
+    (instances
+      (project "TIME II PCB"
+        (path "/ada74dd6-9313-41da-aa43-aea44c6d55c8"
+          (reference "R13") (unit 1)
+        )
+      )
+    )
+  )
   (symbol (lib_name "GND_7") (lib_id "power:GND") (at 124.46 35.56 0) (unit 1)
     (in_bom yes) (on_board yes) (dnp no) (fields_autoplaced)
@@
         )
       )
+    )
+  )
+  (symbol (lib_id "Device:R") (at 391.16 106.68 90) (unit 1)
+    (in_bom yes) (on_board yes) (dnp no) (fields_autoplaced)
+    (property "Reference" "R5" (at 391.16 100.33 90)
+      (effects (font (size 1.27 1.27)))
+    )
+    (property "Value" "R" (at 391.16 102.87 90)
+      (effects (font (size 1.27 1.27)))
+    )
+    (property "Footprint" "" (at 391.16 108.458 90)
+      (effects (font (size 1.27 1.27)) hide)
+    )
+    (property "Datasheet" "~" (at 391.16 106.68 0)
+      (effects (font (size 1.27 1.27)) hide)
+    )
+    (pin "1")
+    (pin "2")
+    (instances
+      (project "TIME II PCB"
+        (path "/ada74dd6-9313-41da-aa43-aea44c6d55c8"
+          (reference "R5") (unit 1)
+        )
+      )
