File: TIME II PCB.kicad_sch (KiCad schematic)
At the start: 75 parts, among them J1 USB_C_Receptacle, J10 Conn_01x02_Male, J11 Conn_01x02_Male, J12 Conn_01x02_Male, J13 Conn_01x03_Male, J14 Conn_01x03_Male, J15 Conn_01x03_Male, J16 Conn_01x03_Male, J17 Conn_01x03_Male, J2 SD_Card, J3 Conn_01x02_Male, J4 Conn_01x02_Male, J5 Conn_01x02_Male, J6 Conn_01x02_Male, J7 Conn_01x02_Male, J8 Conn_01x02_Male, J9 Conn_01x02_Male, Q1 VNP10N07, Q2 VNP10N07, Q3 VNP10N07, Q4 VNP10N07, Q5 VNP10N07, SW1 PTS647SM38SMTR2LFS, SW2 PTS647SM38SMTR2LFS, U1 ESP32-S2-SOLO

Commit message: Add files via upload
Parts:
- removed J4, J5: Conn_01x02_Male, Connector_PinHeader_2.54mm:PinHeader_1x02_P2.54mm_Vertical, symbol Connector:Conn_01x02_Male
- removed R13, R15, R16, R17: 80k, Resistor_SMD:R_0603_1608Metric, symbol Device:R
- added C20: 47 uF, Capacitor_SMD:C_0402_1005Metric, symbol Device:C
- added C21: 1 uF, Capacitor_SMD:C_0402_1005Metric, symbol Device:C
- added C22, C23: 0.1 uF, Capacitor_SMD:C_0402_1005Metric, symbol Device:C
- added C24, C7: 4.7 uF, Capacitor_SMD:C_0402_1005Metric, symbol Device:C
- added C6: 0.47 uF, Capacitor_SMD:C_0402_1005Metric, symbol Device:C
- added D3: LED, LED_SMD:LED_0603_1608Metric, symbol Device:LED
- added D4: D_Schottky, Diode_SMD:D_0402_1005Metric, symbol Device:D_Schottky
- added D5, D6: D, Diode_SMD:D_0402_1005Metric, symbol Device:D
- added DS1, DS2715: ~, symbol DS2715:DS2715
- added J18, J19, J20, J4, J5: Conn_01x03_Pin, Connector_PinHeader_2.54mm:PinHeader_1x03_P2.54mm_Vertical, symbol Connector:Conn_01x03_Pin
- added J21: Conn_01x02_Male, Connector_PinHeader_2.54mm:PinHeader_1x02_P2.54mm_Vertical, symbol Connector:Conn_01x02_Male
- added MAX2: MAX17610, Connector_PinHeader_2.54mm:PinHeader_1x03_P2.54mm_Vertical, symbol MAX17608:MAX17610
- added Q6: NMOS, Package_TO_SOT_THT:TO-220-2_Horizontal_TabDown, symbol Simulation_SPICE:NMOS
- added Q7: PMOS, Package_TO_SOT_SMD:SOT-23, symbol Simulation_SPICE:PMOS
- added R101, R102, R103, R104, R105, R108, R110, R113: R, Resistor_SMD:R_0402_1005Metric, symbol Device:R
- added R107: 7, Resistor_SMD:R_0402_1005Metric, symbol Device:R
- added R112: 300K, Resistor_SMD:R_0402_1005Metric, symbol Device:R
- added RSETI1: 1.8K, Resistor_SMD:R_0402_1005Metric, symbol Device:R
- C1, C2, C3, C4: footprint Capacitor_SMD:C_0603_1608Metric -> Capacitor_SMD:C_0402_1005Metric
- C10, C8: renamed from C?; footprint Capacitor_SMD:C_0603_1608Metric -> Capacitor_SMD:C_0402_1005Metric
- C11, C13, C9: renamed from C?; footprint (none) -> Capacitor_SMD:C_0402_1005Metric
- C12, C14: renamed from C?; value .1uF -> 47uF; footprint Capacitor_SMD:C_0603_1608Metric -> Capacitor_SMD:C_0402_1005Metric
- L1: renamed from L?; value 4.7uH -> 2.2uH; footprint Inductor_SMD:L_0603_1608Metric_Pad1.05x0.95mm_HandSolder -> Connector_PinHeader_2.54mm:PinHeader_1x03_P2.54mm_Vertical
- R1, R10, R11, R12, R18, R19, R20, R21, R22, R3, R6, R7, R8, R9: footprint Resistor_SMD:R_0603_1608Metric -> Resistor_SMD:R_0402_1005Metric
- R14: value 80k -> 150K; footprint Resistor_SMD:R_0603_1608Metric -> Resistor_SMD:R_0402_1005Metric
- R15, R24, R25, R26, R27, R28, R29, R30: renamed from R?; footprint (none) -> Resistor_SMD:R_0402_1005Metric
- R16: renamed from R?; value 10.2k -> 15.2k; footprint Resistor_SMD:R_0603_1608Metric_Pad0.98x0.95mm_HandSolder -> Resistor_SMD:R_0402_1005Metric
- R17: renamed from R?; value 56k -> 10.2k; footprint Resistor_SMD:R_0603_1608Metric_Pad0.98x0.95mm_HandSolder -> Resistor_SMD:R_0402_1005Metric
- R23, R31, R32: renamed from R?; footprint Resistor_SMD:R_0603_1608Metric_Pad0.98x0.95mm_HandSolder -> Resistor_SMD:R_0402_1005Metric
- gave numbers to parts that had none: 4
Connections:
- net USB_P is gone; now on net GND: F1.2, R15.1, R24.1, U3.1 (V1)
- net 5v: now also J18.3 (Pin_3), J19.3 (Pin_3), J20.3 (Pin_3), J4.3 (Pin_3), J5.3 (Pin_3); no longer R14.1
- net GND: now also R14.2, C20.2, C21.2, C22.2, C6.1, C6.2, C7.1, C7.2, D6.1 (K), D6.2 (A), DS1.11 (SNS+), J18.1 (Pin_1), J19.1 (Pin_1), J20.1 (Pin_1), J4.1 (Pin_1), J5.1 (Pin_1), MAX2.1 (IN), MAX2.12 (OUT), MAX2.7 (GND), MAX2.8 (SETI), R107.1, RSETI1.1, RSETI1.2; no longer J3.1 (Pin_1), J6.1 (Pin_1), J7.1 (Pin_1)
- net therm_1: now also J18.2 (Pin_2); no longer J3.2 (Pin_2)
- net therm_2: now also J4.2 (Pin_2)
- net therm_3: now also J5.2 (Pin_2)
- net therm_4: now also J19.2 (Pin_2); no longer J6.2 (Pin_2)
- net therm_5: now also J20.2 (Pin_2); no longer J7.2 (Pin_2), R14.2
- new net: J6.2 (Pin_2), J7.1 (Pin_1)
- new net: J21.1 (Pin_1), J7.2 (Pin_2)
- new net: C24.2, DS1.2 (Vch), Q7.2 (G), R103.2
- new net: DS1.16 (Vbatt), R112.2, R113.1
- new net: C23.2, DS1.12 (SNS-), DS1.3 (VSS), DS1.8 (CTG), DS1.9 (Mode), J3.1 (Pin_1), J6.1 (Pin_1), Q6.3 (S), R107.2, R108.2, R113.2
- new net: MAX2.6 (CLMODE), R14.1
- new net: Q6.1 (D), R105.1
- new net: DS1.14 (Rt), R105.2
- new net: C23.1, DS1.1 (Cbias)
- new net: C22.1, DS1.13 (Vdd), R101.2
- new net: D3.1 (K), R104.1
- new net: DS1.4 (LED1), R104.2
- new net: D5.1 (K), R102.1
- new net: DS1.10 (Div), R110.1
- new net: DS1.15 (THM), J3.2 (Pin_2), R110.2
- new net: J21.2 (Pin_2), Q7.1 (D), R102.2, R112.1
- new net: Q6.2 (G), R108.1
- new net 6V DC: D4.2 (A)
- new net LOAD: C20.1, C21.1, C24.1, D3.2 (A), D4.1 (K), D5.2 (A), Q7.3 (S), R101.1, R103.1

Commit message: layout
Parts:
- removed J10, J11, J12, J6, J7, J8, J9: Conn_01x02_Male, Connector_PinHeader_2.54mm:PinHeader_1x02_P2.54mm_Vertical, symbol Connector:Conn_01x02_Male
- removed J13, J14, J15, J16, J17: Conn_01x03_Male, Connector_PinHeader_2.54mm:PinHeader_1x03_P2.54mm_Vertical, symbol Connector:Conn_01x03_Male
- removed J18, J19, J20, J4, J5: Conn_01x03_Pin, Connector_PinHeader_2.54mm:PinHeader_1x03_P2.54mm_Vertical, symbol Connector:Conn_01x03_Pin
- removed R20, R22: 1.5k, Resistor_SMD:R_0402_1005Metric, symbol Device:R
- added J4, J5, J6, J7, J8: Conn_01x05_Pin, Connector_JST:JST_XH_B5B-XH-AM_1x05_P2.50mm_Vertical, symbol Connector:Conn_01x05_Pin
- added R13, R5: 1.5k, Resistor_SMD:R_0402_1005Metric, symbol Device:R
- added R2: 100K, Resistor_SMD:R_0402_1005Metric, symbol Device:R
- added R4: 100k, Resistor_SMD:R_0402_1005Metric, symbol Device:R
- DS1: footprint (none) -> Package_SO:SOIC-16_3.9x9.9mm_P1.27mm
- F1: footprint (none) -> Fuse:Fuse_0603_1608Metric
- J1: footprint usb:USB4105-GF-A -> usb:USB4120-03-C_GCT
- J2: footprint (none) -> sdcard:MEM2075-00-140-01-A_GCT
- J21, J3: footprint Connector_PinHeader_2.54mm:PinHeader_1x02_P2.54mm_Vertical -> Connector_JST:JST_XH_B2B-XH-AM_1x02_P2.50mm_Vertical
- L1: footprint Connector_PinHeader_2.54mm:PinHeader_1x03_P2.54mm_Vertical -> inductor:IND_B1047AS-2R2N=P3
- MAX2: footprint Connector_PinHeader_2.54mm:PinHeader_1x03_P2.54mm_Vertical -> Package_DFN_QFN:WDFN-12-1EP_3x3mm_P0.45mm_EP1.7x2.5mm
- Q1, Q2, Q3, Q4, Q5: footprint Package_TO_SOT_THT:TO-220-3_Vertical -> Package_TO_SOT_SMD:SOT-23-3
- Q6: footprint Package_TO_SOT_THT:TO-220-2_Horizontal_TabDown -> Package_TO_SOT_SMD:SOT-23-3
- Q7: footprint Package_TO_SOT_SMD:SOT-23 -> Package_TO_SOT_SMD:SOT-23-3
- SW1, SW2: footprint footprints:PTS647SM38SMTR2LFS -> button:SW_PTS647SM38SMTR2LFS_CNK
- U2: footprint adp2303:ADP2303ARDZ-3.3-R7 -> Package_SO:SOIC-8-N7_3.9x4.9mm_P1.27mm
- U3: footprint MSE_12_ADI -> Package_SO:MSOP-12-1EP_3x4mm_P0.65mm_EP1.65x2.85mm
Connections:
- net 6V DC is gone; now on net 5v: D4.2 (A)
- net 5v: now also J4.5 (Pin_5), J5.5 (Pin_5), J6.5 (Pin_5), J7.5 (Pin_5), J8.5 (Pin_5)
- net BAT: now also J21.2 (Pin_2), Q7.1 (D), R102.2, R112.1, R2.1
- net GND: now also J2.12 (SHELL1), J2.13 (SHELL2), J4.1 (Pin_1), J5.1 (Pin_1), J6.1 (Pin_1), J7.1 (Pin_1), J8.1 (Pin_1), R4.2; no longer C6.1, C7.1, D6.1 (K), F1.2, MAX2.1 (IN), MAX2.12 (OUT), MAX2.8 (SETI), R15.1, R24.1, RSETI1.1, SW2.1, U3.1 (V1)
- net SERVO_1: now also U1.19 (GPIO11/TOUCH11/ADC2_CH0/FSPID/FSPIIO5), J4.2 (Pin_2)
- net SERVO_2: now also U1.21 (GPIO13/TOUCH13/ADC2_CH2/FSPIQ/FSPIIO7), J5.2 (Pin_2)
- net SERVO_3: now also J8.2 (Pin_2)
- net SERVO_4: now also J7.2 (Pin_2)
- net SERVO_5: now also J6.2 (Pin_2)
- net V_MON: now also R2.2, R4.1
- net heater_1: now also SW2.4, U1.38 (GPIO2/TOUCH2/ADC1_CH1), U1.39 (GPIO1/TOUCH1/ADC1_CH0), R5.2
- net heater_3: now also R19.2, U1.34 (MTDI/GPIO41/CLK_OUT1)
- net heater_4: now also U1.26 (GPIO45)
- net heater_5: now also U1.37 (U0TXD/GPIO43/CLK_OUT1), R13.2; no longer R19.2
- net therm_1: now also U1.35 (MTMS/GPIO42), J4.4 (Pin_4)
- net therm_2: now also U1.15 (GPIO3/TOUCH3/ADC1_CH2), J5.4 (Pin_4)
- net therm_3: now also U1.17 (GPIO9/TOUCH9/ADC1_CH8/FSPIHD), J8.4 (Pin_4)
- net therm_4: now also U1.4 (GPIO4/TOUCH4/ADC1_CH3), J7.4 (Pin_4)
- net therm_5: now also U1.23 (GPIO21), J6.4 (Pin_4)
- net at Q3.1 (G): now also R18.1
- net at J21.1 (Pin_1): now also C23.2, DS1.12 (SNS-), DS1.3 (VSS), DS1.8 (CTG), DS1.9 (Mode), J3.1 (Pin_1), Q6.3 (S), R107.2, R108.2, R113.2
- net at Q5.2 (D): now also J8.3 (Pin_3)
- net at Q2.2 (D): now also J6.3 (Pin_3)
- net at Q3.2 (D): now also J7.3 (Pin_3)
- net at Q5.1 (G): now also R19.1
- net at Q1.1 (G): now also R5.1; no longer R18.1
- net at Q1.2 (D): now also J5.3 (Pin_3)
- net at Q2.1 (G): now also R13.1; no longer R19.1
- net at Q4.2 (D): now also J4.3 (Pin_3)
- new net: MAX2.8 (SETI), RSETI1.1
- new net OR Gate: C7.1, D6.1 (K), MAX2.12 (OUT), R15.1, R24.1, U3.1 (V1)
- new net USB_P: C6.1, F1.2, MAX2.1 (IN)
Other:
- note added: "CONNECTORS"
- note removed: "Heaters"
- note removed: "SERVO OUTPUT"
- note removed: "Thermistors"
- moved on the sheet: C20, C21, C22, C23, C24, D3, D4, D5, DS1, J21, J3, Q4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

Commit message: motor driver
Parts:
- removed J4, J5, J6, J7, J8: Conn_01x05_Pin, Connector_JST:JST_XH_B5B-XH-AM_1x05_P2.50mm_Vertical, symbol Connector:Conn_01x05_Pin
- added C15, C17, C25: 10uF, Capacitor_SMD:C_0402_1005Metric, symbol Device:C
- added C16, C18, C26: 0.01uF, Capacitor_SMD:C_0402_1005Metric, symbol Device:C
- added C19, C27, C5: 2.2pF, Capacitor_SMD:C_0402_1005Metric, symbol Device:C
- added J4, J5, J6, J7, J8: Conn_01x06_Pin, Connectors_JST:JST_XH_B06B-XH-A_06x2.50mm_Straight, symbol Connector:Conn_01x06_Pin
- added R20: 10k, Resistor_SMD:R_0402_1005Metric, symbol Device:R
- added R22, R33: .33, Resistor_SMD:R_0402_1005Metric, symbol Device:R
- added R25.5: 2k, Resistor_SMD:R_0402_1005Metric, symbol Device:R
- added SW3, SW4, SW5, SW6, SW7: SW_SPDT, Connector_PinHeader_1.27mm:PinHeader_1x03_P1.27mm_Vertical, symbol Switch:SW_SPDT
- added U4, U5, U6: ~, Package_DFN_QFN:QFN-16-1EP_3x3mm_P0.5mm_EP1.7x1.7mm, symbol DRV883:DRV883
- J1: footprint usb:USB4120-03-C_GCT -> usb:USB4105-GF-A
- R10, R11, R12, R9: value 10k -> .33
- R25: value 156k -> 154k
Connections:
- net OR Gate is gone; now on net 5v: C7.1, D6.1 (K), MAX2.12 (OUT), R15.1, R24.1, U3.1 (V1)
- net 3v3: now also R20.1; no longer R10.1, R11.1, R12.1, R9.1, U1.2 (3V3)
- net 5v: now also C10.1, MAX2.8 (SETI), Q6.2 (G), R108.1, R28.2, R29.1, RSETI1.1, U2.1 (BST), U3.10 (V2UV), J4.5 (Pin_5), J5.5 (Pin_5), J6.5 (Pin_5), J7.5 (Pin_5), J8.5 (Pin_5); no longer U3.2 (V2TEST)
- net GND: now also C4.1, R10.2, R11.2, R12.2, R9.2, SW2.1, U3.13 (EPAD), C15.2, C17.2, C19.2, C25.2, C27.2, C5.2, J4.1 (Pin_1), J5.1 (Pin_1), J6.1 (Pin_1), J7.1 (Pin_1), J8.1 (Pin_1), R22.2, R33.2, U4.13 (GND), U5.13 (GND), U6.13 (GND); no longer C4.2, U3.EPAD
- net MISO: now also J2.2 (CMD), U1.22 (GPIO14/TOUCH14/ADC2_CH3/FSPIWP/FSPIDQS); no longer J2.7 (DAT0), R12.2
- net MOSI: now also J2.7 (DAT0), U1.18 (GPIO10/TOUCH10/ADC1_CH9/FSPICS0/FSPIIO4); no longer J2.2 (CMD), R10.2
- net SCK: now also U1.19 (GPIO11/TOUCH11/ADC2_CH0/FSPID/FSPIIO5); no longer R11.2
- net SERVO_1: now also U1.11 (GPIO18/U1RXD/ADC2_CH7/DAC_2/CLK_OUT3), SW3.3 (C), U4.16 (AIN1); no longer U1.19 (GPIO11/TOUCH11/ADC2_CH0/FSPID/FSPIIO5)
- net SERVO_2: now also U1.12 (GPIO8/TOUCH8/ADC1_CH7), SW5.3 (C), U4.9 (BIN1); no longer U1.21 (GPIO13/TOUCH13/ADC2_CH2/FSPIQ/FSPIIO7)
- net SERVO_3: now also SW6.3 (C), U5.16 (AIN1)
- net SERVO_4: now also SW4.3 (C), U5.9 (BIN1)
- net SERVO_5: now also SW7.3 (C), U6.16 (AIN1), U6.9 (BIN1)
- net SS: now also U1.23 (GPIO21); no longer R9.2
- net heater_1: no longer R5.2, SW2.4, U1.38 (GPIO2/TOUCH2/ADC1_CH1)
- net heater_3: now also U1.10 (GPIO17/U1TXD/ADC2_CH6/DAC_1); no longer U1.34 (MTDI/GPIO41/CLK_OUT1)
- net heater_4: now also U1.21 (GPIO13/TOUCH13/ADC2_CH2/FSPIQ/FSPIIO7); no longer U1.26 (GPIO45)
- net heater_5: now also U1.26 (GPIO45); no longer U1.37 (U0TXD/GPIO43/CLK_OUT1)
- net therm_1: now also U1.4 (GPIO4/TOUCH4/ADC1_CH3), J4.4 (Pin_4); no longer U1.35 (MTMS/GPIO42)
- net therm_2: now also J5.4 (Pin_4)
- net therm_3: now also J6.4 (Pin_4)
- net therm_4: now also U1.16 (GPIO46), J7.4 (Pin_4); no longer U1.4 (GPIO4/TOUCH4/ADC1_CH3)
- net therm_5: now also U1.20 (GPIO12/TOUCH12/ADC2_CH1/FSPICLK/FSPIIO6), J8.4 (Pin_4); no longer U1.23 (GPIO21)
- net at Q5.2 (D): now also J6.3 (Pin_3)
- net at SW2.3, U1.27 (GPIO0): now also C4.2; no longer C4.1
- net at C23.2, DS1.12 (SNS-), DS1.3 (VSS)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: no longer DS1.9 (Mode)
- net at Q6.1 (D), R105.1: now also C22.1, R101.2
- net at R105.2: now also DS1.13 (Vdd); no longer DS1.14 (Rt)
- net at Q4.2 (D): now also J4.3 (Pin_3)
- net at Q1.2 (D): now also J5.3 (Pin_3)
- net at R27.1, U3.8 (V2OK): now also R30.2, U3.6 (CMPOUT1)
- net at C23.1: now also DS1.9 (Mode); no longer DS1.1 (Cbias)
- net at Q3.2 (D): now also J7.3 (Pin_3)
- net at Q2.2 (D): now also J8.3 (Pin_3)
- net at J3.2 (Pin_2), R110.2: no longer DS1.15 (THM)
- net SERVO_3A: now reaches U1.24 (SPIIO4/GPIO33/FSPIHD)
- net SERVO_3A: now also U5.15 (AIN2)
- net SERVO_4A: now reaches U1.25 (SPIIO5/GPIO34/FSPICS0)
- net SERVO_4A: now also U5.10 (BIN2)
- net SERVO_5A: now reaches U1.28 (SPIIO6/GPIO35/FSPID)
- net SERVO_5A: now also U6.10 (BIN2), U6.15 (AIN2)
- net SERVO_1A: now reaches U1.6 (GPIO6/TOUCH6/ADC1_CH5)
- net SERVO_1A: now also U4.15 (AIN2)
- net SERVO_2A: now reaches U1.7 (GPIO7/TOUCH7/ADC1_CH6)
- net SERVO_2A: now also U4.10 (BIN2)
- net MOT_CON: now reaches U1.9 (GPIO16/U0CTS/ADC2_CH5/XTAL_32K_N)
- net MOT_CON: now also U4.1 (NSLEEP), U5.1 (NSLEEP), U6.1 (NSLEEP)
- new net: C26.2, U6.11 (VCP)
- new net: C25.1, C26.1, U6.12 (VM)
- new net: R33.1, U6.3 (AISEN)
- new net: R22.1, U6.6 (BISEN)
- new net: C27.1, U6.8 (NFAULT)
- new net: C16.2, U4.11 (VCP)
- new net: C15.1, C16.1, U4.12 (VM)
- new net: R9.1, U4.3 (AISEN)
- new net: R10.1, U4.6 (BISEN)
- new net: C5.1, U4.8 (NFAULT)
- new net: C18.2, U5.11 (VCP)
- new net: C17.1, C18.1, U5.12 (VM)
- new net: R12.1, U5.3 (AISEN)
- new net: R11.1, U5.6 (BISEN)
- new net: C19.1, U5.8 (NFAULT)
- new net: R20.2, SW2.4
- new net: R25.2, R25.5.1
- new net: R25.5.2, R26.1
- new net ACTUATOR_1: J4.2 (Pin_2), SW3.2 (B)
- new net ACTUATOR_2: J5.2 (Pin_2), SW5.2 (B)
- new net ACTUATOR_3: J6.2 (Pin_2), SW6.2 (B)
- new net ACTUATOR_4: J7.2 (Pin_2), SW4.2 (B)
- new net ACTUATOR_5: J8.2 (Pin_2), SW7.2 (B)
- new net MOTOR_1: SW3.1 (A), U4.2 (AOUT1)
- new net MOTOR_1A: J4.6 (Pin_6), U4.4 (AOUT2)
- new net MOTOR_2: SW5.1 (A), U4.7 (BOUT1)
- new net MOTOR_2A: J5.6 (Pin_6), U4.5 (BOUT2)
- new net MOTOR_3: SW6.1 (A), U5.2 (AOUT1)
- new net MOTOR_3A: J6.6 (Pin_6), U5.4 (AOUT2)
- new net MOTOR_4: SW4.1 (A), U5.7 (BOUT1)
- new net MOTOR_4A: J7.6 (Pin_6), U5.5 (BOUT2)
- new net MOTOR_5: SW7.1 (A), U6.2 (AOUT1), U6.7 (BOUT1)
- new net MOTOR_5A: J8.6 (Pin_6), U6.4 (AOUT2), U6.5 (BOUT2)
- new net MOT_MON_1: U4.14 (VINT)
- new net MOT_MON_2: U5.14 (VINT)
- new net MOT_MON_3: U6.14 (VINT)
- new net heater_2: R5.2, U1.38 (GPIO2/TOUCH2/ADC1_CH1)
- now unconnected: U3.3 (CMP1)
Other:
- moved on the sheet: C1, C10, C11, C12, C13, C2, C20, C21, C22, C23, C24, C3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

Commit message: done?
Parts:
- removed R105: R, Resistor_SMD:R_0402_1005Metric, symbol Device:R
- added R34: 86K, Resistor_SMD:R_0402_1005Metric, symbol Device:R
- R101: value R -> 150
- R102: value R -> 220
- R103, R104: value R -> 470
- R107: value 7 -> .25
- R108, R110: value R -> 10K
- R113: value R -> 100K
Connections:
- net MISO: now also U1.35 (MTMS/GPIO42); no longer U1.22 (GPIO14/TOUCH14/ADC2_CH3/FSPIWP/FSPIDQS)
- net MOSI: now also U1.32 (MTCK/GPIO39/CLK_OUT3); no longer U1.18 (GPIO10/TOUCH10/ADC1_CH9/FSPICS0/FSPIIO4)
- net SCK: now also U1.33 (MTDO/GPIO40/CLK_OUT2); no longer U1.19 (GPIO11/TOUCH11/ADC2_CH0/FSPID/FSPIIO5)
- net SERVO_2A: now also U1.8 (GPIO15/U0RTS/ADC2_CH4/XTAL_32K_P); no longer U1.7 (GPIO7/TOUCH7/ADC1_CH6)
- net SERVO_3A: now also U1.18 (GPIO10/TOUCH10/ADC1_CH9/FSPICS0/FSPIIO4); no longer U1.24 (SPIIO4/GPIO33/FSPIHD)
- net SERVO_4A: now also U1.17 (GPIO9/TOUCH9/ADC1_CH8/FSPIHD); no longer U1.25 (SPIIO5/GPIO34/FSPICS0)
- net SERVO_5A: now also U1.22 (GPIO14/TOUCH14/ADC2_CH3/FSPIWP/FSPIDQS); no longer U1.28 (SPIIO6/GPIO35/FSPID)
- net SS: now also U1.34 (MTDI/GPIO41/CLK_OUT1); no longer U1.23 (GPIO21)
- net V_MON: now also U1.7 (GPIO7/TOUCH7/ADC1_CH6); no longer U1.8 (GPIO15/U0RTS/ADC2_CH4/XTAL_32K_P)
- net heater_4: now also U1.25 (SPIIO5/GPIO34/FSPICS0); no longer U1.21 (GPIO13/TOUCH13/ADC2_CH2/FSPIQ/FSPIIO7)
- net heater_5: now also U1.21 (GPIO13/TOUCH13/ADC2_CH2/FSPIQ/FSPIIO7); no longer U1.26 (GPIO45)
- net therm_3: now also U1.19 (GPIO11/TOUCH11/ADC2_CH0/FSPID/FSPIIO5); no longer U1.17 (GPIO9/TOUCH9/ADC1_CH8/FSPIHD)
- net therm_4: no longer U1.16 (GPIO46)
- net therm_5: now also U1.24 (SPIIO4/GPIO33/FSPIHD); no longer U1.20 (GPIO12/TOUCH12/ADC2_CH1/FSPICLK/FSPIIO6)
- net at C22.1, R101.2: now also DS1.13 (Vdd); no longer Q6.1 (D)
- net at R25.5.2, R26.1: now also U3.3 (CMP1)
- net at DS1.14 (Rt): now also R34.2
- net at DS1.15 (THM): now also J3.2 (Pin_2), R110.2
- new net: Q6.1 (D), R34.1

Commit message: main (old rev) local changes push
Connections:
- net 5v: now also U3.2 (V2TEST); no longer C7.1, D6.1 (K), MAX2.12 (OUT), MAX2.8 (SETI), R15.1, R24.1, RSETI1.1, U3.1 (V1)
- net USB_P: now also MAX2.2 (IN)
- new net OR Gate: C7.1, D6.1 (K), MAX2.12 (OUT), MAX2.8 (SETI), R15.1, R24.1, RSETI1.1, U3.1 (V1)
Changed lines of the file:
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@@
   (junction (at 104.14 231.14) (diameter 0) (color 0 0 0 0)
   )
-  (junction (at 111.76 231.14) (diameter 0) (color 0 0 0 0)
-  )
   (junction (at 416.56 261.62) (diameter 0) (color 0 0 0 0)
   )
@@
   (junction (at 200.66 170.18) (diameter 0) (color 0 0 0 0)
   )
+  (junction (at 281.94 233.68) (diameter 0) (color 0 0 0 0)
+  )
   (junction (at 309.88 101.6) (diameter 0) (color 0 0 0 0)
   )
@@
     (stroke (width 0) (type default))
   )
-  (wire (pts (xy 111.76 228.6) (xy 111.76 231.14))
+  (wire (pts (xy 281.94 233.68) (xy 281.94 236.22))
     (stroke (width 0) (type default))
   )
@@
     (stroke (width 0) (type default))
   )
+  (wire (pts (xy 111.76 228.6) (xy 110.49 228.6))
+    (stroke (width 0) (type default))
+  )
   (wire (pts (xy 182.88 154.94) (xy 182.88 160.02))
     (stroke (width 0) (type default))
@@
     (stroke (width 0) (type default))
   )
+  (wire (pts (xy 110.49 228.6) (xy 110.49 233.68))
+    (stroke (width 0) (type default))
+  )
   (wire (pts (xy 101.6 322.58) (xy 101.6 330.2))
     (stroke (width 0) (type default))
@@
     (stroke (width 0) (type default))
   )
+  (wire (pts (xy 110.49 233.68) (xy 111.76 233.68))
+    (stroke (width 0) (type default))
+  )
   (wire (pts (xy 584.2 222.25) (xy 590.55 222.25))
     (stroke (width 0) (type default))
@@
   )
   (symbol (lib_id "Device:R") (at 170.18 237.49 0) (unit 1)
-    (in_bom yes) (on_board yes) (dnp no) (fields_autoplaced)
+    (in_bom yes) (on_board yes) (dnp no)
     (property "Reference" "R28" (at 172.72 236.2199 0)
       (effects (font (size 1.27 1.27)) (justify left))
