File: TIME II PCB.kicad_sch (KiCad schematic)
At the start: 65 parts, among them J1 SD_Card, J2 USB_C_Receptacle, J3 Conn_01x06, J4 Conn_01x06, J5 Conn_01x06, J6 Conn_01x02_Male, J7 Conn_01x02_Male, J8 Conn_01x02_Pin, Q1 VNP10N07, Q2 VNP10N07, Q3 VNP10N07, SW1 SW_SPDT, U1 STM32F103C8Tx, U2 LTC4420CMSE-PBF, U5 AMS1117-3.3, Y1 16 khz

Commit message: sd card update
Connections:
- net SS renamed CD
Changed lines of the file:
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@@
 	(global_label "3v3"
 		(shape input)
-		(at 86.36 20.32 90)
-		(fields_autoplaced yes)
-		(effects
-			(font
-				(size 1.27 1.27)
-			)
-			(justify left)
-		)
-		(property "Intersheetrefs" "${INTERSHEET_REFS}"
-			(at 86.36 13.9482 90)
-			(effects
-				(font
-					(size 1.27 1.27)
-				)
-				(justify left)
+		(at 86.36 20.32 270)
+		(fields_autoplaced yes)
+		(effects
+			(font
+				(size 1.27 1.27)
+			)
+			(justify right)
+		)
+		(property "Intersheetrefs" "${INTERSHEET_REFS}"
+			(at 86.36 26.6918 90)
+			(effects
+				(font
+					(size 1.27 1.27)
+				)
+				(justify right)
 				(hide yes)
 			)
@@
 		)
 	)
-	(global_label "SS"
+	(global_label "CD"
 		(shape input)
 		(at 62.23 97.79 180)
@@
 		)
 		(property "Intersheetrefs" "${INTERSHEET_REFS}"
-			(at 56.8258 97.79 0)
+			(at 56.7048 97.79 0)
 			(effects
 				(font
@@
 		)
 	)
-	(global_label "SS"
+	(global_label "CD"
 		(shape input)
 		(at 193.04 48.26 270)
@@
 		)
 		(property "Intersheetrefs" "${INTERSHEET_REFS}"
-			(at 193.04 53.6642 90)
-			(effects
-				(font
+			(at 193.04 53.7852 90)
+			(effects
+				(font
